File: USB_POWERED_v2.sch (EAGLE design)
At the start: 16 parts, among them J1 USB

Commit message: update routing. Will probably change again before file is sent...
Parts:
- R1: device ERIC:RESISTOR_ARRAY_2 -> ERIC:RESISTOR_ARRAY_4CTS_742
Changed lines of the file:
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@@
 <part name="U$2" library="HARWIN" deviceset="M06" device=""/>
 <part name="R6" library="ERIC" deviceset="RESISTOR_ARRAY_2" device="" value="1K"/>
-<part name="R1" library="ERIC" deviceset="RESISTOR_ARRAY_2" device="" value="27"/>
+<part name="R1" library="ERIC" deviceset="RESISTOR_ARRAY_4" device="CTS_742" value="27"/>
 </parts>
 <sheets>
